Commit message: xacro update finish->joint_state pub&sub configuring...

File: src/surgical_robot_control/urdf/surgical_tool_right.urdf.xacro (robot description, xacro)
@@ -3,4 +3,5 @@
 <!-- <xacro:include filename="my_materials.xacro"/> -->
 <!-- <xacro:include filename="./colors.urdf.xacro" /> -->
+<xacro:property name="robot_name" value="right"/>
 <xacro:property name="width" value="0.05"/>
 <xacro:property name="height" value="0.2"/>
@@ -15,16 +16,49 @@
 <xacro:property name="blue" value="0 0 0.8 1"/>
 <xacro:property name="blueviolet" value="0.54 0.16 0.88 1.0"/>
-    <link name="base_surgical_robot">
+    <link name="${robot_name}/base">
         <inertial>
             <origin xyz="0.0 0.0 0.0" rpy="0.0 0.0 0.0"/>
-            <!-- <inertia ixx="1.0" ixy="0.0" ixz="0.0" iyy="1.0" iyz="0.0" izz="1.0"/> -->
+            <inertia ixx="1.0" ixy="0.0" ixz="0.0" iyy="1.0" iyz="0.0" izz="1.0"/>
+            <mass value="${mass}"/>
         </inertial>
     </link>
-    <joint name="base-shaft" type="fixed">
+    <joint name="${robot_name}/base-actuator" type="revolute">
+        <origin xyz="0.0 0.0 0.0" rpy="0.0 0.0 0.0"/>
+        <parent link="${robot_name}/base"/>
+        <child link="${robot_name}/actuator"/>
+        <axis xyz="1.0 0.0 0.0"/>
+        <limit lower="-3.14" upper="3.14" effort="30" velocity="1"/>
+    </joint>
+    <link name="${robot_name}/actuator">
+        <!-- <inertial>
+            <origin xyz="0.0 0.0 0.0" rpy="0.0 0.0 0.0"/>
+            <mesh filename="package://surgical_robot_control/meshes/ActuatorModule_Blender_zero.dae"/>
+            <mass value="${mass}"/>
+            <inertia ixx="${mass/12*(width*width+width*width)}" ixy="0.0" ixz="0.0"
+                iyy="${mass/12*(width*width+width*width)}" iyz="0.0"
+                izz="${mass/12*(height*height+height*height)}"/>
+        </inertial> -->
+        <visual>
+            <origin xyz="0.0 0.0 0.0" rpy="0.0 0.0 0.0"/>
+            <geometry>
+                <mesh filename="package://surgical_robot_control/meshes/ActuatorModule_Blender_zero.dae"/>
+            </geometry>
+            <!-- <material name="actuator">
+                <color rgba="1.0 1.0 0.0 0.4"/>
+            </material> -->
+        </visual>
+        <collision>
+            <origin xyz="0.0 0.0 0.0" rpy="0.0 0.0 0.0"/>
+            <geometry>
+                <mesh filename="package://surgical_robot_control/meshes/ActuatorModule_Blender_zero.dae"/>
+            </geometry>
+        </collision>
+    </link>
+    <joint name="${robot_name}/actuator-shaft" type="fixed">
         <origin xyz="0.187 0.0 0.0" rpy="0.0 0.0 0.0"/>
-        <parent link="base_surgical_robot"/>
-        <child link="shaft"/>
-    </joint>
-    <link name="shaft">
+        <parent link="${robot_name}/actuator"/>
+        <child link="${robot_name}/shaft"/>
+    </joint>
+    <link name="${robot_name}/shaft">
         <inertial>
             <origin xyz="0.25 0.0 0.0" rpy="0.0 2.0 0.0"/>
@@ -39,5 +73,5 @@
                 <cylinder radius="0.0015" length="${height}"/>
             </geometry>
-            <material name="link3">
+            <material name="${robot_name}/shaft">
                 <color rgba="1.0 1.0 0.0 0.3"/>
             </material>
@@ -50,72 +84,72 @@
         </collision>
     </link>
-    <joint name="tilt-1" type="revolute">
+    <joint name="${robot_name}/tilt-1" type="revolute">
         <origin xyz="${height} 0.0 0.0" rpy="0.0 0.0 0.0"/>
-        <parent link="shaft"/>
-        <child link="seg_tilt-1"/>
-        <axis xyz="${tilt}"/>
-        <limit lower="-0.7854" upper="0.7854" effort="30.0" velocity="3.141"/>
-    </joint>
-    <link name="seg_tilt-1">
-        <visual>
-            <origin xyz="0.0 0.0 0.0" rpy="0.0 0.0 0.0"/>
-            <geometry>
-                <mesh filename="package://surgical_robot_control/meshes/continuum_segment_Blender_zero_lightgreen.dae" scale="0.001 0.001 0.001"/>
-            </geometry>
-        </visual>
-    </link>
-    <joint name="pan-1" type="revolute">
-        <origin xyz="${seg_interval} 0.0 0.0" rpy="0.0 0.0 0.0"/>
-        <parent link="seg_tilt-1"/>
-        <child link="seg_pan-1"/>
-        <axis xyz="${pan}"/>
-        <limit lower="-0.7854" upper="0.7854" effort="30.0" velocity="3.141"/>
-    </joint>
-    <link name="seg_pan-1">
-        <visual>
-            <origin xyz="0.0 0.0 0.0" rpy="1.5708 0.0 0.0"/>
-            <geometry>
-                <mesh filename="package://surgical_robot_control/meshes/continuum_segment_Blender_zero_violet.dae" scale="0.001 0.001 0.001"/>
-            </geometry>
-        </visual>
-    </link>
-    <joint name="tilt-2" type="revolute">
-        <origin xyz="${seg_interval} 0.0 0.0" rpy="0.0 0.0 0.0"/>
-        <parent link="seg_pan-1"/>
-        <child link="seg_tilt-2"/>
-        <axis xyz="${tilt}"/>
-        <limit lower="-0.7854" upper="0.7854" effort="30.0" velocity="3.141"/>
-    </joint>
-    <link name="seg_tilt-2">
-        <visual>
-            <origin xyz="0.0 0.0 0.0" rpy="0.0 0.0 0.0"/>
-            <geometry>
-                <mesh filename="package://surgical_robot_control/meshes/continuum_segment_Blender_zero_lightgreen.dae" scale="0.001 0.001 0.001"/>
-            </geometry>
-        </visual>
-    </link>
-    <joint name="pan-2" type="revolute">
-        <origin xyz="${seg_interval} 0.0 0.0" rpy="0.0 0.0 0.0"/>
-        <parent link="seg_tilt-2"/>
-        <child link="seg_pan-2"/>
-        <axis xyz="${pan}"/>
-        <limit lower="-0.7854" upper="0.7854" effort="30.0" velocity="3.141"/>
-    </joint>
-    <link name="seg_pan-2">
-        <visual>
-            <origin xyz="0.0 0.0 0.0" rpy="1.5708 0.0 0.0"/>
-            <geometry>
-                <mesh filename="package://surgical_robot_control/meshes/continuum_segment_Blender_zero_violet.dae" scale="0.001 0.001 0.001"/>
-            </geometry>
-        </visual>
-    </link>
-    <joint name="tilt-3" type="revolute">
-        <origin xyz="${seg_interval} 0.0 0.0" rpy="0.0 0.0 0.0"/>
-        <parent link="seg_pan-2"/>
-        <child link="seg_tilt-3"/>
-        <axis xyz="${tilt}"/>
-        <limit lower="-0.7854" upper="0.7854" effort="30.0" velocity="3.141"/>
-    </joint>
-    <link name="seg_tilt-3">
+        <parent link="${robot_name}/shaft"/>
+        <child link="${robot_name}/seg_tilt-1"/>
+        <axis xyz="${tilt}"/>
+        <limit lower="-0.7854" upper="0.7854" effort="30.0" velocity="3.141"/>
+    </joint>
+    <link name="${robot_name}/seg_tilt-1">
+        <visual>
+            <origin xyz="0.0 0.0 0.0" rpy="0.0 0.0 0.0"/>
+            <geometry>
+                <mesh filename="package://surgical_robot_control/meshes/continuum_segment_Blender_zero_lightgreen.dae" scale="0.001 0.001 0.001"/>
+            </geometry>
+        </visual>
+    </link>
+    <joint name="${robot_name}/pan-1" type="revolute">
+        <origin xyz="${seg_interval} 0.0 0.0" rpy="0.0 0.0 0.0"/>
+        <parent link="${robot_name}/seg_tilt-1"/>
+        <child link="${robot_name}/seg_pan-1"/>
+        <axis xyz="${pan}"/>
+        <limit lower="-0.7854" upper="0.7854" effort="30.0" velocity="3.141"/>
+    </joint>
+    <link name="${robot_name}/seg_pan-1">
+        <visual>
+            <origin xyz="0.0 0.0 0.0" rpy="1.5708 0.0 0.0"/>
+            <geometry>
+                <mesh filename="package://surgical_robot_control/meshes/continuum_segment_Blender_zero_violet.dae" scale="0.001 0.001 0.001"/>
+            </geometry>
+        </visual>
+    </link>
+    <joint name="${robot_name}/tilt-2" type="revolute">
+        <origin xyz="${seg_interval} 0.0 0.0" rpy="0.0 0.0 0.0"/>
+        <parent link="${robot_name}/seg_pan-1"/>
+        <child link="${robot_name}/seg_tilt-2"/>
+        <axis xyz="${tilt}"/>
+        <limit lower="-0.7854" upper="0.7854" effort="30.0" velocity="3.141"/>
+    </joint>
+    <link name="${robot_name}/seg_tilt-2">
+        <visual>
+            <origin xyz="0.0 0.0 0.0" rpy="0.0 0.0 0.0"/>
+            <geometry>
+                <mesh filename="package://surgical_robot_control/meshes/continuum_segment_Blender_zero_lightgreen.dae" scale="0.001 0.001 0.001"/>
+            </geometry>
+        </visual>
+    </link>
+    <joint name="${robot_name}/pan-2" type="revolute">
+        <origin xyz="${seg_interval} 0.0 0.0" rpy="0.0 0.0 0.0"/>
+        <parent link="${robot_name}/seg_tilt-2"/>
+        <child link="${robot_name}/seg_pan-2"/>
+        <axis xyz="${pan}"/>
+        <limit lower="-0.7854" upper="0.7854" effort="30.0" velocity="3.141"/>
+    </joint>
+    <link name="${robot_name}/seg_pan-2">
+        <visual>
+            <origin xyz="0.0 0.0 0.0" rpy="1.5708 0.0 0.0"/>
+            <geometry>
+                <mesh filename="package://surgical_robot_control/meshes/continuum_segment_Blender_zero_violet.dae" scale="0.001 0.001 0.001"/>
+            </geometry>
+        </visual>
+    </link>
+    <joint name="${robot_name}/tilt-3" type="revolute">
+        <origin xyz="${seg_interval} 0.0 0.0" rpy="0.0 0.0 0.0"/>
+        <parent link="${robot_name}/seg_pan-2"/>
+        <child link="${robot_name}/seg_tilt-3"/>
+        <axis xyz="${tilt}"/>
+        <limit lower="-0.7854" upper="0.7854" effort="30.0" velocity="3.141"/>
+    </joint>
+    <link name="${robot_name}/seg_tilt-3">
         <visual>
             <origin xyz="0.0 0.0 0.0" rpy="0.0 0.0 0.0"/>
@@ -127,10 +161,10 @@
     <joint name="pan-3" type="revolute">
         <origin xyz="${seg_interval} 0.0 0.0" rpy="0.0 0.0 0.0"/>
-        <parent link="seg_tilt-3"/>
-        <child link="seg_pan-3"/>
-        <axis xyz="${pan}"/>
-        <limit lower="-0.7854" upper="0.7854" effort="30.0" velocity="3.141"/>
-    </joint>
-    <link name="seg_pan-3">
+        <parent link="${robot_name}/seg_tilt-3"/>
+        <child link="${robot_name}/seg_pan-3"/>
+        <axis xyz="${pan}"/>
+        <limit lower="-0.7854" upper="0.7854" effort="30.0" velocity="3.141"/>
+    </joint>
+    <link name="${robot_name}/seg_pan-3">
         <visual>
             <origin xyz="0.0 0.0 0.0" rpy="1.5708 0.0 0.0"/>
@@ -142,55 +176,55 @@
     <joint name="tilt-4" type="revolute">
         <origin xyz="${seg_interval} 0.0 0.0" rpy="0.0 0.0 0.0"/>
-        <parent link="seg_pan-3"/>
-        <child link="seg_tilt-4"/>
-        <axis xyz="${tilt}"/>
-        <limit lower="-0.7854" upper="0.7854" effort="30.0" velocity="3.141"/>
-    </joint>
-    <link name="seg_tilt-4">
-        <visual>
-            <origin xyz="0.0 0.0 0.0" rpy="0.0 0.0 0.0"/>
-            <geometry>
-                <mesh filename="package://surgical_robot_control/meshes/continuum_segment_Blender_zero_lightgreen.dae" scale="0.001 0.001 0.001"/>
-            </geometry>
-        </visual>
-    </link>
-    <joint name="pan-4" type="revolute">
-        <origin xyz="${seg_interval} 0.0 0.0" rpy="0.0 0.0 0.0"/>
-        <parent link="seg_tilt-4"/>
-        <child link="seg_pan-4"/>
-        <axis xyz="${pan}"/>
-        <limit lower="-0.7854" upper="0.7854" effort="30.0" velocity="3.141"/>
-    </joint>
-    <link name="seg_pan-4">
-        <visual>
-            <origin xyz="0.0 0.0 0.0" rpy="1.5708 0.0 0.0"/>
-            <geometry>
-                <mesh filename="package://surgical_robot_control/meshes/continuum_segment_Blender_zero_violet.dae" scale="0.001 0.001 0.001"/>
-            </geometry>
-        </visual>
-    </link>
-    <joint name="tilt-5" type="revolute">
-        <origin xyz="${seg_interval} 0.0 0.0" rpy="0.0 0.0 0.0"/>
-        <parent link="seg_pan-4"/>
-        <child link="seg_tilt-5"/>
-        <axis xyz="${tilt}"/>
-        <limit lower="-0.7854" upper="0.7854" effort="30.0" velocity="3.141"/>
-    </joint>
-    <link name="seg_tilt-5">
-        <visual>
-            <origin xyz="0.0 0.0 0.0" rpy="0.0 0.0 0.0"/>
-            <geometry>
-                <mesh filename="package://surgical_robot_control/meshes/continuum_segment_Blender_zero_lightgreen.dae" scale="0.001 0.001 0.001"/>
-            </geometry>
-        </visual>
-    </link>
-    <joint name="pan-5" type="revolute">
-        <origin xyz="${seg_interval} 0.0 0.0" rpy="0.0 0.0 0.0"/>
-        <parent link="seg_tilt-5"/>
-        <child link="seg_pan-5"/>
-        <axis xyz="${pan}"/>
-        <limit lower="-0.7854" upper="0.7854" effort="30.0" velocity="3.141"/>
-    </joint>
-    <link name="seg_pan-5">
+        <parent link="${robot_name}/seg_pan-3"/>
+        <child link="${robot_name}/seg_tilt-4"/>
+        <axis xyz="${tilt}"/>
+        <limit lower="-0.7854" upper="0.7854" effort="30.0" velocity="3.141"/>
+    </joint>
+    <link name="${robot_name}/seg_tilt-4">
+        <visual>
+            <origin xyz="0.0 0.0 0.0" rpy="0.0 0.0 0.0"/>
+            <geometry>
+                <mesh filename="package://surgical_robot_control/meshes/continuum_segment_Blender_zero_lightgreen.dae" scale="0.001 0.001 0.001"/>
+            </geometry>
+        </visual>
+    </link>
+    <joint name="${robot_name}/pan-4" type="revolute">
+        <origin xyz="${seg_interval} 0.0 0.0" rpy="0.0 0.0 0.0"/>
+        <parent link="${robot_name}/seg_tilt-4"/>
+        <child link="${robot_name}/seg_pan-4"/>
+        <axis xyz="${pan}"/>
+        <limit lower="-0.7854" upper="0.7854" effort="30.0" velocity="3.141"/>
+    </joint>
+    <link name="${robot_name}/seg_pan-4">
+        <visual>
+            <origin xyz="0.0 0.0 0.0" rpy="1.5708 0.0 0.0"/>
+            <geometry>
+                <mesh filename="package://surgical_robot_control/meshes/continuum_segment_Blender_zero_violet.dae" scale="0.001 0.001 0.001"/>
+            </geometry>
+        </visual>
+    </link>
+    <joint name="${robot_name}/tilt-5" type="revolute">
+        <origin xyz="${seg_interval} 0.0 0.0" rpy="0.0 0.0 0.0"/>
+        <parent link="${robot_name}/seg_pan-4"/>
+        <child link="${robot_name}/seg_tilt-5"/>
+        <axis xyz="${tilt}"/>
+        <limit lower="-0.7854" upper="0.7854" effort="30.0" velocity="3.141"/>
+    </joint>
+    <link name="${robot_name}/seg_tilt-5">
+        <visual>
+            <origin xyz="0.0 0.0 0.0" rpy="0.0 0.0 0.0"/>
+            <geometry>
+                <mesh filename="package://surgical_robot_control/meshes/continuum_segment_Blender_zero_lightgreen.dae" scale="0.001 0.001 0.001"/>
+            </geometry>
+        </visual>
+    </link>
+    <joint name="${robot_name}/pan-5" type="revolute">
+        <origin xyz="${seg_interval} 0.0 0.0" rpy="0.0 0.0 0.0"/>
+        <parent link="${robot_name}/seg_tilt-5"/>
+        <child link="${robot_name}/seg_pan-5"/>
+        <axis xyz="${pan}"/>
+        <limit lower="-0.7854" upper="0.7854" effort="30.0" velocity="3.141"/>
+    </joint>
+    <link name="${robot_name}/seg_pan-5">
         <visual>
             <origin xyz="0.0 0.0 0.0" rpy="1.5708 0.0 0.0"/>

Commit message: simulator update

File: src/surgical_robot_control/urdf/surgical_tool_left.urdf.xacro (robot description, xacro)
@@ -159,5 +159,5 @@
         </visual>
     </link>
-    <joint name="pan-3" type="revolute">
+    <joint name="${robot_name}/pan-3" type="revolute">
         <origin xyz="${seg_interval} 0.0 0.0" rpy="0.0 0.0 0.0"/>
         <parent link="${robot_name}/seg_tilt-3"/>
@@ -174,5 +174,5 @@
         </visual>
     </link>
-    <joint name="tilt-4" type="revolute">
+    <joint name="${robot_name}/tilt-4" type="revolute">
         <origin xyz="${seg_interval} 0.0 0.0" rpy="0.0 0.0 0.0"/>
         <parent link="${robot_name}/seg_pan-3"/>

File: src/surgical_robot_control/urdf/surgical_tool_right.urdf.xacro (robot description, xacro)
@@ -159,5 +159,5 @@
         </visual>
     </link>
-    <joint name="pan-3" type="revolute">
+    <joint name="${robot_name}/pan-3" type="revolute">
         <origin xyz="${seg_interval} 0.0 0.0" rpy="0.0 0.0 0.0"/>
         <parent link="${robot_name}/seg_tilt-3"/>
@@ -174,5 +174,5 @@
         </visual>
     </link>
-    <joint name="tilt-4" type="revolute">
+    <joint name="${robot_name}/tilt-4" type="revolute">
         <origin xyz="${seg_interval} 0.0 0.0" rpy="0.0 0.0 0.0"/>
         <parent link="${robot_name}/seg_pan-3"/>
