Commit message: xacro file update!

File: src/surgical_robot_control/urdf/surgical_tool.urdf.xacro (robot description, xacro)
@@ -2,39 +2,34 @@
 <robot xmlns:xacro="https://www.ros.org/wiki/xacro" name="surgical_robot_control">
 <!-- <xacro:include filename="my_materials.xacro"/> -->
+<!-- <xacro:include filename="./colors.urdf.xacro" /> -->
 <xacro:property name="width" value="0.05"/>
 <xacro:property name="height" value="0.2"/>
 <xacro:property name="mass" value="0.1"/>
-    <link name="base_link">
+<!-- segment macro -->
+<xacro:property name="seg_interval" value="0.0018"/>
+<xacro:property name="tilt" value="0.0 1.0 0.0"/>
+<xacro:property name="pan" value="0.0 0.0 1.0"/>
+<xacro:property name="gray" value="1.0 1.0 1.0 0.4"/>
+<xacro:property name="black" value="0.0 0.0 0.0 1.0"/>
+<xacro:property name="orange" value="1.0 0.4 0.0 1.0"/>
+<xacro:property name="blue" value="0 0 0.8 1"/>
+<xacro:property name="blueviolet" value="0.54 0.16 0.88 1.0"/>
+    <link name="base_surgical_robot">
         <inertial>
-            <origin xyz="0.0 0.0 ${height/2}" rpy="0.0 0.0 0.0"/>
-            <mass value="${mass}"/>
-            <inertia ixx="1.0" ixy="0.0" ixz="0.0" iyy="1.0" iyz="0.0" izz="1.0"/>
+            <origin xyz="0.0 0.0 0.0" rpy="0.0 0.0 0.0"/>
+            <!-- <inertia ixx="1.0" ixy="0.0" ixz="0.0" iyy="1.0" iyz="0.0" izz="1.0"/> -->
         </inertial>
-        <visual>
-            <origin xyz="0.0 0.0 ${height/2}" rpy="0.0 0.0 0.0"/>
-            <geometry>
-                <box size="${width} ${width} ${height}"/>
-            </geometry>
-            <material name="base_link">
-                <color rgba="1.0 0.0 0.0 1.0"/>
-            </material>
-        </visual>
-        <collision>
-            <origin xyz="0.0 0.0 ${height/2}" rpy="0.0 0.0 0.0"/>
-            <geometry>
-                <box size="${width} ${width} ${height}"/>
-            </geometry>
-        </collision>
-    </link>
-    <joint name="Joint1" type="revolute">
-        <origin xyz="0.0 0.0 0.25" rpy="0.0 0.0 0.0"/>
-        <parent link="base_link"/>
-        <child link="Link1"/>
+    </link>
+    <joint name="base-actuator" type="revolute">
+        <origin xyz="0.0 0.0 0.0" rpy="0.0 0.0 0.0"/>
+        <parent link="base_surgical_robot"/>
+        <child link="actuator"/>
         <axis xyz="1.0 0.0 0.0"/>
         <limit lower="-3.14" upper="3.14" effort="30" velocity="1"/>
     </joint>
-    <link name="Link1">
+    <link name="actuator">
         <inertial>
-            <origin xyz="0.0 0.0 ${height/2}" rpy="0.0 0.0 0.0"/>
+            <origin xyz="0.0 0.0 0.0" rpy="0.0 0.0 0.0"/>
+            <mesh filename="package://surgical_robot_control/meshes/ActuatorModule_Blender_zero.dae"/>
             <mass value="${mass}"/>
             <inertia ixx="${mass/12*(width*width+width*width)}" ixy="0.0" ixz="0.0"
@@ -43,29 +38,27 @@
         </inertial>
         <visual>
-            <origin xyz="0.0 0.0 ${height/2}" rpy="0.0 0.0 0.0"/>
-            <geometry>
-                <box size="${width} ${width} ${height}"/>
-            </geometry>
-            <material name="link1">
-                <color rgba="0.0 1.0 0.0 1.0"/>
-            </material>
+            <origin xyz="0.0 0.0 0.0" rpy="0.0 0.0 0.0"/>
+            <geometry>
+                <mesh filename="package://surgical_robot_control/meshes/ActuatorModule_Blender_zero.dae"/>
+            </geometry>
+            <!-- <material name="actuator">
+                <color rgba="1.0 1.0 0.0 0.4"/>
+            </material> -->
         </visual>
         <collision>
-            <origin xyz="0.0 0.0 ${height/2}" rpy="0.0 0.0 0.0"/>
-            <geometry>
-                <box size="${width} ${width} ${height}"/>
+            <origin xyz="0.0 0.0 0.0" rpy="0.0 0.0 0.0"/>
+            <geometry>
+                <mesh filename="package://surgical_robot_control/meshes/ActuatorModule_Blender_zero.dae"/>
             </geometry>
         </collision>
     </link>
-    <joint name="Joint2" type="revolute">
-        <origin xyz="0.0 0.0 0.25" rpy="0.0 0.0 0.0"/>
-        <parent link="Link1"/>
-        <child link="Link2"/>
-        <axis xyz="1.0 0.0 0.0"/>
-        <limit lower="-3.14" upper="3.14" effort="30" velocity="1"/>
-    </joint>
-    <link name="Link2">
+    <joint name="actuator-shaft" type="fixed">
+        <origin xyz="0.187 0.0 0.0" rpy="0.0 0.0 0.0"/>
+        <parent link="actuator"/>
+        <child link="shaft"/>
+    </joint>
+    <link name="shaft">
         <inertial>
-            <origin xyz="0.0 0.0 ${height/2}" rpy="0.0 0.0 0.0"/>
+            <origin xyz="0.25 0.0 0.0" rpy="0.0 2.0 0.0"/>
             <mass value="${mass}"/>
             <inertia ixx="${mass/12*(width*width+width*width)}" ixy="0.0" ixz="0.0"
@@ -74,49 +67,168 @@
         </inertial>
         <visual>
-            <origin xyz="0.0 0.0 ${height/2}" rpy="0.0 0.0 0.0"/>
-            <geometry>
-                <box size="${width} ${width} ${height}"/>
-            </geometry>
-            <material name="link2">
-                <color rgba="0.0 0.0 1.0 1.0"/>
+            <origin xyz="${height/2} 0.0 0.0" rpy="0.0 1.5708 0.0"/>
+            <geometry>
+                <cylinder radius="0.0015" length="${height}"/>
+            </geometry>
+            <material name="link3">
+                <color rgba="1.0 1.0 0.0 0.3"/>
             </material>
         </visual>
         <collision>
-            <origin xyz="0.0 0.0 ${height/2}" rpy="0.0 0.0 0.0"/>
-            <geometry>
-                <box size="${width} ${width} ${height}"/>
+            <origin xyz="${height/2} 0.0 0.0" rpy="0.0 0.0 0.0"/>
+            <geometry>
+                <cylinder radius="0.0015" length="${height}"/>
             </geometry>
         </collision>
     </link>
-    <joint name="Joint3" type="revolute">
-        <origin xyz="0.0 0.0 0.25" rpy="0.0 0.0 0.0"/>
-        <parent link="Link2"/>
-        <child link="Link3"/>
-        <axis xyz="1.0 0.0 0.0"/>
-        <limit lower="-3.14" upper="3.14" effort="30" velocity="1"/>
-    </joint>
-    <link name="Link3">
-        <inertial>
-            <origin xyz="0.0 0.0 ${height/2}" rpy="0.0 0.0 0.0"/>
-            <mass value="${mass}"/>
-            <inertia ixx="${mass/12*(width*width+width*width)}" ixy="0.0" ixz="0.0"
-                iyy="${mass/12*(width*width+width*width)}" iyz="0.0"
-                izz="${mass/12*(height*height+height*height)}"/>
-        </inertial>
-        <visual>
-            <origin xyz="0.0 0.0 ${height/2}" rpy="0.0 0.0 0.0"/>
-            <geometry>
-                <box size="${width} ${width} ${height}"/>
-            </geometry>
-            <material name="link3">
-                <color rgba="0.0 1.0 1.0 1.0"/>
-            </material>
-        </visual>
-        <collision>
-            <origin xyz="0.0 0.0 ${height/2}" rpy="0.0 0.0 0.0"/>
-            <geometry>
-                <box size="${width} ${width} ${height}"/>
-            </geometry>
-        </collision>
+    <joint name="tilt-1" type="revolute">
+        <origin xyz="${height} 0.0 0.0" rpy="0.0 0.0 0.0"/>
+        <parent link="shaft"/>
+        <child link="seg_tilt-1"/>
+        <axis xyz="${tilt}"/>
+        <limit lower="-0.7854" upper="0.7854" effort="30.0" velocity="3.141"/>
+    </joint>
+    <link name="seg_tilt-1">
+        <visual>
+            <origin xyz="0.0 0.0 0.0" rpy="0.0 0.0 0.0"/>
+            <geometry>
+                <mesh filename="package://surgical_robot_control/meshes/continuum_segment_Blender_zero_lightgreen.dae" scale="0.001 0.001 0.001"/>
+            </geometry>
+        </visual>
+    </link>
+    <joint name="pan-1" type="revolute">
+        <origin xyz="${seg_interval} 0.0 0.0" rpy="0.0 0.0 0.0"/>
+        <parent link="seg_tilt-1"/>
+        <child link="seg_pan-1"/>
+        <axis xyz="${pan}"/>
+        <limit lower="-0.7854" upper="0.7854" effort="30.0" velocity="3.141"/>
+    </joint>
+    <link name="seg_pan-1">
+        <visual>
+            <origin xyz="0.0 0.0 0.0" rpy="1.5708 0.0 0.0"/>
+            <geometry>
+                <mesh filename="package://surgical_robot_control/meshes/continuum_segment_Blender_zero_violet.dae" scale="0.001 0.001 0.001"/>
+            </geometry>
+        </visual>
+    </link>
+    <joint name="tilt-2" type="revolute">
+        <origin xyz="${seg_interval} 0.0 0.0" rpy="0.0 0.0 0.0"/>
+        <parent link="seg_pan-1"/>
+        <child link="seg_tilt-2"/>
+        <axis xyz="${tilt}"/>
+        <limit lower="-0.7854" upper="0.7854" effort="30.0" velocity="3.141"/>
+    </joint>
+    <link name="seg_tilt-2">
+        <visual>
+            <origin xyz="0.0 0.0 0.0" rpy="0.0 0.0 0.0"/>
+            <geometry>
+                <mesh filename="package://surgical_robot_control/meshes/continuum_segment_Blender_zero_lightgreen.dae" scale="0.001 0.001 0.001"/>
+            </geometry>
+        </visual>
+    </link>
+    <joint name="pan-2" type="revolute">
+        <origin xyz="${seg_interval} 0.0 0.0" rpy="0.0 0.0 0.0"/>
+        <parent link="seg_tilt-2"/>
+        <child link="seg_pan-2"/>
+        <axis xyz="${pan}"/>
+        <limit lower="-0.7854" upper="0.7854" effort="30.0" velocity="3.141"/>
+    </joint>
+    <link name="seg_pan-2">
+        <visual>
+            <origin xyz="0.0 0.0 0.0" rpy="1.5708 0.0 0.0"/>
+            <geometry>
+                <mesh filename="package://surgical_robot_control/meshes/continuum_segment_Blender_zero_violet.dae" scale="0.001 0.001 0.001"/>
+            </geometry>
+        </visual>
+    </link>
+    <joint name="tilt-3" type="revolute">
+        <origin xyz="${seg_interval} 0.0 0.0" rpy="0.0 0.0 0.0"/>
+        <parent link="seg_pan-2"/>
+        <child link="seg_tilt-3"/>
+        <axis xyz="${tilt}"/>
+        <limit lower="-0.7854" upper="0.7854" effort="30.0" velocity="3.141"/>
+    </joint>
+    <link name="seg_tilt-3">
+        <visual>
+            <origin xyz="0.0 0.0 0.0" rpy="0.0 0.0 0.0"/>
+            <geometry>
+                <mesh filename="package://surgical_robot_control/meshes/continuum_segment_Blender_zero_lightgreen.dae" scale="0.001 0.001 0.001"/>
+            </geometry>
+        </visual>
+    </link>
+    <joint name="pan-3" type="revolute">
+        <origin xyz="${seg_interval} 0.0 0.0" rpy="0.0 0.0 0.0"/>
+        <parent link="seg_tilt-3"/>
+        <child link="seg_pan-3"/>
+        <axis xyz="${pan}"/>
+        <limit lower="-0.7854" upper="0.7854" effort="30.0" velocity="3.141"/>
+    </joint>
+    <link name="seg_pan-3">
+        <visual>
+            <origin xyz="0.0 0.0 0.0" rpy="1.5708 0.0 0.0"/>
+            <geometry>
+                <mesh filename="package://surgical_robot_control/meshes/continuum_segment_Blender_zero_violet.dae" scale="0.001 0.001 0.001"/>
+            </geometry>
+        </visual>
+    </link>
+    <joint name="tilt-4" type="revolute">
+        <origin xyz="${seg_interval} 0.0 0.0" rpy="0.0 0.0 0.0"/>
+        <parent link="seg_pan-3"/>
+        <child link="seg_tilt-4"/>
+        <axis xyz="${tilt}"/>
+        <limit lower="-0.7854" upper="0.7854" effort="30.0" velocity="3.141"/>
+    </joint>
+    <link name="seg_tilt-4">
+        <visual>
+            <origin xyz="0.0 0.0 0.0" rpy="0.0 0.0 0.0"/>
+            <geometry>
+                <mesh filename="package://surgical_robot_control/meshes/continuum_segment_Blender_zero_lightgreen.dae" scale="0.001 0.001 0.001"/>
+            </geometry>
+        </visual>
+    </link>
+    <joint name="pan-4" type="revolute">
+        <origin xyz="${seg_interval} 0.0 0.0" rpy="0.0 0.0 0.0"/>
+        <parent link="seg_tilt-4"/>
+        <child link="seg_pan-4"/>
+        <axis xyz="${pan}"/>
+        <limit lower="-0.7854" upper="0.7854" effort="30.0" velocity="3.141"/>
+    </joint>
+    <link name="seg_pan-4">
+        <visual>
+            <origin xyz="0.0 0.0 0.0" rpy="1.5708 0.0 0.0"/>
+            <geometry>
+                <mesh filename="package://surgical_robot_control/meshes/continuum_segment_Blender_zero_violet.dae" scale="0.001 0.001 0.001"/>
+            </geometry>
+        </visual>
+    </link>
+    <joint name="tilt-5" type="revolute">
+        <origin xyz="${seg_interval} 0.0 0.0" rpy="0.0 0.0 0.0"/>
+        <parent link="seg_pan-4"/>
+        <child link="seg_tilt-5"/>
+        <axis xyz="${tilt}"/>
+        <limit lower="-0.7854" upper="0.7854" effort="30.0" velocity="3.141"/>
+    </joint>
+    <link name="seg_tilt-5">
+        <visual>
+            <origin xyz="0.0 0.0 0.0" rpy="0.0 0.0 0.0"/>
+            <geometry>
+                <mesh filename="package://surgical_robot_control/meshes/continuum_segment_Blender_zero_lightgreen.dae" scale="0.001 0.001 0.001"/>
+            </geometry>
+        </visual>
+    </link>
+    <joint name="pan-5" type="revolute">
+        <origin xyz="${seg_interval} 0.0 0.0" rpy="0.0 0.0 0.0"/>
+        <parent link="seg_tilt-5"/>
+        <child link="seg_pan-5"/>
+        <axis xyz="${pan}"/>
+        <limit lower="-0.7854" upper="0.7854" effort="30.0" velocity="3.141"/>
+    </joint>
+    <link name="seg_pan-5">
+        <visual>
+            <origin xyz="0.0 0.0 0.0" rpy="1.5708 0.0 0.0"/>
+            <geometry>
+                <mesh filename="package://surgical_robot_control/meshes/continuum_segment_Blender_zero_violet.dae" scale="0.001 0.001 0.001"/>
+            </geometry>
+        </visual>
     </link>
 </robot>

File: src/surgical_robot_control/urdf/surgical_tool_v1.urdf (robot description, URDF)
Before this commit: robot surgical_robot, 13 links, 12 joints
Links:
- link seg_pan5: geometry collision cylinder length=0.003 radius=0.003; visual mesh filename=package://surgical_robot_control/meshes/ActuatorModule.stl scale=0.001 0.001 0.001
